File: hardware/drone-pcb/mcu.kicad_sch (KiCad schematic)
At the start: 27 parts, among them J1 USB-C, J5 DEBUG, SW1 BOOT, SW2 RESET, U1 ESP32-S3-WROOM-1-N8R2, U22 USBLC6-2SC6

Commit message: G3 draft: PCB layouts for all four boards (routing incomplete), stop at G3
- Flight controller (6 layers, D-062), 4-in-1 ESC (4 layers, 180-degree
  channel copies, D-063) and both ToF satellites laid out by Python scripts
  in tools/pcb (KiCad 7 + Freerouting 1.9 + a grid finishing router, D-064).
- ToF satellites fully routed, DRC 0. FC has 29 and ESC 51 open connections,
  listed in review/G3/open-connections.md (OQ-19). ESC motor-phase copper is
  too narrow and needs a power-stage rework before G4.
- Slimmer connectors (D-061) revise the G2 schematics; outlines and the
  16 x 25 mm mounting pattern per D-060.
- G3 package: layer plots, 3D renders, DRC reports, stackup, IPC-2221 widths
  with measured copper, antenna/USB/IMU notes, autorouted nets.
- Mass budget 86.2 g (measured outline areas, 6-layer FC); SDK and Flight Lab
  parameters, figures, banner and explorer regenerated.

STATUS: DRAFT - UNVERIFIED - requires human review at Gate G3

Co-Authored-By: Claude Opus 5.5 <noreply@anthropic.com>
Claude-Session: https://claude.ai/code/session_01Vd9yCNNEC59Q8t73ayFh14
Parts:
- J5: footprint Connector_PinHeader_1.27mm:PinHeader_1x06_P1.27mm_Vertical -> microscout:PadRow_1x06_P1.50mm_SMD
- SW1, SW2: footprint Button_Switch_SMD:SW_Push_1P1T_XKB_TS-1187A -> Button_Switch_SMD:SW_Push_1P1T_NO_CK_KMR2; LCSC C318884 -> (none); MPN TS-1187A-B-A-B -> KMR211NGLFS (C&K) or KMR2-footprint equivalent; Note (none) -> D-061: 4.2x2.8 mm switch; LCSC number UNCONFIRMED
Other:
- note added: "Debug pads (UART0 ROM log, EN, IO0) - SMD"
- note added: "pads, nothing fitted"
- note removed: "Debug pads (UART0 ROM log, EN, IO0) - optional 1.27 mm"
- note removed: "header, not fitted"
Changed lines of the file:
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@@
   (title_block
     (title "MicroScout flight controller - MCU and USB")
-    (date "2026-10-08")
+    (date "2026-10-09")
     (rev "G2-draft-1")
     (company "MicroScout (open hardware, CERN-OHL-S-2.0)")
@@
         (font (size 1.27 1.27))
         (justify left bottom)))
-    (property "Footprint" "Button_Switch_SMD:SW_Push_1P1T_XKB_TS-1187A"
+    (property "Footprint" "Button_Switch_SMD:SW_Push_1P1T_NO_CK_KMR2"
       (at 40.64 139.7 0)
       (effects
@@
       (effects
         (font (size 1.27 1.27)) hide))
-    (property "LCSC" "C318884"
+    (property "MPN" "KMR211NGLFS (C&K) or KMR2-footprint equivalent"
       (at 40.64 139.7 0)
       (effects
         (font (size 1.27 1.27)) hide))
-    (property "MPN" "TS-1187A-B-A-B"
+    (property "Note" "D-061: 4.2x2.8 mm switch; LCSC number UNCONFIRMED"
       (at 40.64 139.7 0)
       (effects
@@
         (font (size 1.27 1.27))
         (justify left bottom)))
-    (property "Footprint" "Button_Switch_SMD:SW_Push_1P1T_XKB_TS-1187A"
+    (property "Footprint" "Button_Switch_SMD:SW_Push_1P1T_NO_CK_KMR2"
       (at 78.74 139.7 0)
       (effects
@@
       (effects
         (font (size 1.27 1.27)) hide))
-    (property "LCSC" "C318884"
+    (property "MPN" "KMR211NGLFS (C&K) or KMR2-footprint equivalent"
       (at 78.74 139.7 0)
       (effects
         (font (size 1.27 1.27)) hide))
-    (property "MPN" "TS-1187A-B-A-B"
+    (property "Note" "D-061: 4.2x2.8 mm switch; LCSC number UNCONFIRMED"
       (at 78.74 139.7 0)
       (effects
@@
       (justify right bottom))
 )
-  (text "Debug pads (UART0 ROM log, EN, IO0) - optional 1.27 mm"
+  (text "Debug pads (UART0 ROM log, EN, IO0) - SMD"
     (at 271.644 33.48 0)
     (effects
@@
       (justify left bottom))
 )
-  (text "header, not fitted"
+  (text "pads, nothing fitted"
     (at 271.644 36.68 0)
     (effects
@@
         (font (size 1.27 1.27))
         (justify left bottom)))
-    (property "Footprint" "Connector_PinHeader_1.27mm:PinHeader_1x06_P1.27mm_Vertical"
+    (property "Footprint" "microscout:PadRow_1x06_P1.50mm_SMD"
       (at 289.56 50.8 0)
       (effects
