File: hardware/drone-pcb/power.kicad_sch (KiCad schematic)
At the start: 81 parts, among them J2 XT30PW-M, J6 JST-XH 3 (balance), J7 ESC link (JST-SH 8), J8 ESC VBAT pad, J9 ESC GND pad, Q5 AO3400A, SW3 POWER, U2 BQ25887, U23 TLV6700, U24 TPS22810, U25 MT3608, U3 TPS62162, U4 TPS62133, U8 LTC2954-1, U9 INA226

Commit message: G3 draft: PCB layouts for all four boards (routing incomplete), stop at G3
- Flight controller (6 layers, D-062), 4-in-1 ESC (4 layers, 180-degree
  channel copies, D-063) and both ToF satellites laid out by Python scripts
  in tools/pcb (KiCad 7 + Freerouting 1.9 + a grid finishing router, D-064).
- ToF satellites fully routed, DRC 0. FC has 29 and ESC 51 open connections,
  listed in review/G3/open-connections.md (OQ-19). ESC motor-phase copper is
  too narrow and needs a power-stage rework before G4.
- Slimmer connectors (D-061) revise the G2 schematics; outlines and the
  16 x 25 mm mounting pattern per D-060.
- G3 package: layer plots, 3D renders, DRC reports, stackup, IPC-2221 widths
  with measured copper, antenna/USB/IMU notes, autorouted nets.
- Mass budget 86.2 g (measured outline areas, 6-layer FC); SDK and Flight Lab
  parameters, figures, banner and explorer regenerated.

STATUS: DRAFT - UNVERIFIED - requires human review at Gate G3

Co-Authored-By: Claude Opus 5.5 <noreply@anthropic.com>
Claude-Session: https://claude.ai/code/session_01Vd9yCNNEC59Q8t73ayFh14
Parts:
- J2: value XT30PW-M -> Battery pigtail (XT30); footprint Connector_AMASS:AMASS_XT30PW-M_1x02_P2.50mm_Horizontal -> microscout:Pigtail_2x_SMD_3x6mm_P4.5mm; LCSC C431092 -> (none); MPN XT30PW-M30.G.Y -> XT30 male plug on 18 AWG silicone lead, ~40 mm (bought, han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; Manufacturer Changzhou Amass -> (none); Note (none) -> D-061: pads instead of a board-mount XT30 (saves ~190 mm2)
- J6: value JST-XH 3 (balance) -> Balance pigtail (JST-XH); footprint Connector_JST:JST_XH_S3B-XH-A_1x03_P2.50mm_Horizontal -> microscout:Pigtail_3x_SMD_1.5x3mm_P2.5mm; LCSC C157928 -> (none); MPN S3B-XH-A(LF)(SN) -> JST-XH 3-pin socket on 26 AWG lead, ~40 mm (bought, hand-so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; Note Pin 1 pack -, pin 2 mid, pin 3 pack + left open (UNCONFIRME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 -> D-061: pads instead of a board-mount JST-XH. Pad 1 pack -, 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
- J8, J9: footprint Connector_Wire:SolderWirePad_1x01_SMD_5x10mm -> microscout:Pad_SMD_3x6mm; Note 20 AWG wire to ESC board; pad size set at G3 -> 20 AWG wire to ESC board (3x6 mm pad, D-061)
- SW3: footprint Button_Switch_SMD:SW_Push_1P1T_XKB_TS-1187A -> Button_Switch_SMD:SW_Push_1P1T_NO_CK_KMR2; LCSC C318884 -> (none); MPN TS-1187A-B-A-B -> KMR211NGLFS (C&K) or KMR2-footprint equivalent; Note (none) -> D-061: 4.2x2.8 mm switch; LCSC number UNCONFIRMED
Other:
- note added: "Battery input and current sense (D-035: no fuse, no reverse FET; keyed XT30 on a"
- note added: "Pigtail pad 1 = pack + (red), pad 2 = pack - (black); the keyed XT30 plug is on the 18 AWG lead."
- note added: "pigtail, D-061)"
- note removed: "Battery input and current sense (D-035: no fuse, no reverse FET; keyed XT30)"
- note removed: "XT30 pin 1 = pack +, pin 2 = pack - (footprint polarity to confirm at G3)."
- moved on the sheet: C1, C2, J2, R1, R2, RS1, U9
