File: hardware/drone-pcb/sensors.kicad_sch (KiCad schematic)
At the start: 26 parts, among them J10 Flow deck v2, J11 ToF left, J12 ToF right, J13 ToF rear, J14 ToF front, U10 TCA6408A, U11 TCA6408A, U12 ICM-42688-P, U13 BMP388, U14 QMC5883P

Commit message: G3 draft: PCB layouts for all four boards (routing incomplete), stop at G3
- Flight controller (6 layers, D-062), 4-in-1 ESC (4 layers, 180-degree
  channel copies, D-063) and both ToF satellites laid out by Python scripts
  in tools/pcb (KiCad 7 + Freerouting 1.9 + a grid finishing router, D-064).
- ToF satellites fully routed, DRC 0. FC has 29 and ESC 51 open connections,
  listed in review/G3/open-connections.md (OQ-19). ESC motor-phase copper is
  too narrow and needs a power-stage rework before G4.
- Slimmer connectors (D-061) revise the G2 schematics; outlines and the
  16 x 25 mm mounting pattern per D-060.
- G3 package: layer plots, 3D renders, DRC reports, stackup, IPC-2221 widths
  with measured copper, antenna/USB/IMU notes, autorouted nets.
- Mass budget 86.2 g (measured outline areas, 6-layer FC); SDK and Flight Lab
  parameters, figures, banner and explorer regenerated.

STATUS: DRAFT - UNVERIFIED - requires human review at Gate G3

Co-Authored-By: Claude Opus 5.5 <noreply@anthropic.com>
Claude-Session: https://claude.ai/code/session_01Vd9yCNNEC59Q8t73ayFh14
Parts:
- J10: footprint Connector_PinHeader_1.27mm:PinHeader_1x08_P1.27mm_Vertical -> microscout:PadRow_1x08_P1.50mm_SMD
- J11, J12, J13: footprint Connector_PinHeader_1.27mm:PinHeader_1x05_P1.27mm_Vertical -> microscout:PadRow_1x05_P1.50mm_SMD; Note Solder pads for a 5-wire flex/cable; footprint set at G3 -> SMD solder pads, 1.5 mm pitch (D-061)
- J14: footprint Connector_PinHeader_1.27mm:PinHeader_1x06_P1.27mm_Vertical -> microscout:PadRow_1x06_P1.50mm_SMD; Note Solder pads for a 6-wire flex/cable; footprint set at G3 -> SMD solder pads, 1.5 mm pitch (D-061)
Changed lines of the file:
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@@
   (title_block
     (title "MicroScout flight controller - Sensors and expanders")
-    (date "2026-10-08")
+    (date "2026-10-09")
     (rev "G2-draft-1")
     (company "MicroScout (open hardware, CERN-OHL-S-2.0)")
@@
         (font (size 1.27 1.27))
         (justify left bottom)))
-    (property "Footprint" "Connector_PinHeader_1.27mm:PinHeader_1x05_P1.27mm_Vertical"
+    (property "Footprint" "microscout:PadRow_1x05_P1.50mm_SMD"
       (at 38.1 215.9 0)
       (effects
@@
       (effects
         (font (size 1.27 1.27)) hide))
-    (property "Note" "Solder pads for a 5-wire flex/cable; footprint set at G3"
+    (property "Note" "SMD solder pads, 1.5 mm pitch (D-061)"
       (at 38.1 215.9 0)
       (effects
@@
         (font (size 1.27 1.27))
         (justify left bottom)))
-    (property "Footprint" "Connector_PinHeader_1.27mm:PinHeader_1x05_P1.27mm_Vertical"
+    (property "Footprint" "microscout:PadRow_1x05_P1.50mm_SMD"
       (at 66.04 215.9 0)
       (effects
@@
       (effects
         (font (size 1.27 1.27)) hide))
-    (property "Note" "Solder pads for a 5-wire flex/cable; footprint set at G3"
+    (property "Note" "SMD solder pads, 1.5 mm pitch (D-061)"
       (at 66.04 215.9 0)
       (effects
@@
         (font (size 1.27 1.27))
         (justify left bottom)))
-    (property "Footprint" "Connector_PinHeader_1.27mm:PinHeader_1x05_P1.27mm_Vertical"
+    (property "Footprint" "microscout:PadRow_1x05_P1.50mm_SMD"
       (at 91.44 215.9 0)
       (effects
@@
       (effects
         (font (size 1.27 1.27)) hide))
-    (property "Note" "Solder pads for a 5-wire flex/cable; footprint set at G3"
+    (property "Note" "SMD solder pads, 1.5 mm pitch (D-061)"
       (at 91.44 215.9 0)
       (effects
@@
         (font (size 1.27 1.27))
         (justify left bottom)))
-    (property "Footprint" "Connector_PinHeader_1.27mm:PinHeader_1x06_P1.27mm_Vertical"
+    (property "Footprint" "microscout:PadRow_1x06_P1.50mm_SMD"
       (at 116.84 215.9 0)
       (effects
@@
       (effects
         (font (size 1.27 1.27)) hide))
-    (property "Note" "Solder pads for a 6-wire flex/cable; footprint set at G3"
+    (property "Note" "SMD solder pads, 1.5 mm pitch (D-061)"
       (at 116.84 215.9 0)
       (effects
@@
         (font (size 1.27 1.27))
         (justify left bottom)))
-    (property "Footprint" "Connector_PinHeader_1.27mm:PinHeader_1x08_P1.27mm_Vertical"
+    (property "Footprint" "microscout:PadRow_1x08_P1.50mm_SMD"
       (at 157.48 223.52 0)
       (effects
