File: hardware/esc-pcb/power.kicad_sch (KiCad schematic)
At the start: 10 parts, among them J1 FC link (JST-SH 8), J2 VBAT pad, J3 GND pad, U1 TPS62162

Commit message: G3 draft: PCB layouts for all four boards (routing incomplete), stop at G3
- Flight controller (6 layers, D-062), 4-in-1 ESC (4 layers, 180-degree
  channel copies, D-063) and both ToF satellites laid out by Python scripts
  in tools/pcb (KiCad 7 + Freerouting 1.9 + a grid finishing router, D-064).
- ToF satellites fully routed, DRC 0. FC has 29 and ESC 51 open connections,
  listed in review/G3/open-connections.md (OQ-19). ESC motor-phase copper is
  too narrow and needs a power-stage rework before G4.
- Slimmer connectors (D-061) revise the G2 schematics; outlines and the
  16 x 25 mm mounting pattern per D-060.
- G3 package: layer plots, 3D renders, DRC reports, stackup, IPC-2221 widths
  with measured copper, antenna/USB/IMU notes, autorouted nets.
- Mass budget 86.2 g (measured outline areas, 6-layer FC); SDK and Flight Lab
  parameters, figures, banner and explorer regenerated.

STATUS: DRAFT - UNVERIFIED - requires human review at Gate G3

Co-Authored-By: Claude Opus 5.5 <noreply@anthropic.com>
Claude-Session: https://claude.ai/code/session_01Vd9yCNNEC59Q8t73ayFh14
Parts:
- J2, J3: footprint Connector_Wire:SolderWirePad_1x01_SMD_5x10mm -> microscout:Pad_SMD_3x6mm
Changed lines of the file:
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@@
   (title_block
     (title "MicroScout 4-in-1 ESC - Power and link")
-    (date "2026-10-08")
+    (date "2026-10-09")
     (rev "G2-draft-1")
     (company "MicroScout (open hardware, CERN-OHL-S-2.0)")
@@
         (font (size 1.27 1.27))
         (justify left bottom)))
-    (property "Footprint" "Connector_Wire:SolderWirePad_1x01_SMD_5x10mm"
+    (property "Footprint" "microscout:Pad_SMD_3x6mm"
       (at 55.88 50.8 0)
       (effects
@@
         (font (size 1.27 1.27))
         (justify left bottom)))
-    (property "Footprint" "Connector_Wire:SolderWirePad_1x01_SMD_5x10mm"
+    (property "Footprint" "microscout:Pad_SMD_3x6mm"
       (at 71.12 50.8 0)
       (effects
