File: hardware/tof-satellites/front/tof.kicad_sch (KiCad schematic)
At the start: 10 parts, among them J1 to FC, U1 VL53L5CX

Commit message: G3 draft: PCB layouts for all four boards (routing incomplete), stop at G3
- Flight controller (6 layers, D-062), 4-in-1 ESC (4 layers, 180-degree
  channel copies, D-063) and both ToF satellites laid out by Python scripts
  in tools/pcb (KiCad 7 + Freerouting 1.9 + a grid finishing router, D-064).
- ToF satellites fully routed, DRC 0. FC has 29 and ESC 51 open connections,
  listed in review/G3/open-connections.md (OQ-19). ESC motor-phase copper is
  too narrow and needs a power-stage rework before G4.
- Slimmer connectors (D-061) revise the G2 schematics; outlines and the
  16 x 25 mm mounting pattern per D-060.
- G3 package: layer plots, 3D renders, DRC reports, stackup, IPC-2221 widths
  with measured copper, antenna/USB/IMU notes, autorouted nets.
- Mass budget 86.2 g (measured outline areas, 6-layer FC); SDK and Flight Lab
  parameters, figures, banner and explorer regenerated.

STATUS: DRAFT - UNVERIFIED - requires human review at Gate G3

Co-Authored-By: Claude Opus 5.5 <noreply@anthropic.com>
Claude-Session: https://claude.ai/code/session_01Vd9yCNNEC59Q8t73ayFh14
Parts:
- J1: footprint Connector_PinHeader_1.27mm:PinHeader_1x06_P1.27mm_Vertical -> microscout:PadRow_1x06_P1.50mm_SMD
Changed lines of the file:
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@@
   (title_block
     (title "MicroScout ToF front satellite - VL53L5CX satellite")
-    (date "2026-10-08")
+    (date "2026-10-09")
     (rev "G2-draft-1")
     (company "MicroScout (open hardware, CERN-OHL-S-2.0)")
@@
         (font (size 1.27 1.27))
         (justify left bottom)))
-    (property "Footprint" "Connector_PinHeader_1.27mm:PinHeader_1x06_P1.27mm_Vertical"
+    (property "Footprint" "microscout:PadRow_1x06_P1.50mm_SMD"
       (at 50.8 114.3 0)
       (effects
